File: Hardware/Wireless Switch.kicad_pcb (KiCad board)
At the start: 2 copper layers, 27 parts, among them J1 Uploader, J2 DC_INPUT, J3 OUTPUT1, J4 RTC_CON, K1 G3MB-202PDC5, Q1 BC547, SW1 BOOT, SW2 RESET, SW3 MODE, U1 ESP32-WROOM-32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

Commit message: route pcb
Parts:
- added D2: 1N4148, Diode_THT:D_5W_P10.16mm_Horizontal, F.Cu at (98.0, 65.3)
- added J5: AC_INPUT, TerminalBlock:TerminalBlock_Wuerth_691311400102_P7.62mm, F.Cu at (93.2, 93.7)
- C4: footprint Capacitor_SMD:CP_Elec_4x3.9 -> custom-footprint:CP_Radial_Tantal_D5.0mm_P2.50mm
- C5: value 10uf -> 22uf; footprint Capacitor_SMD:CP_Elec_4x3.9 -> custom-footprint:CP_Radial_Tantal_D5.0mm_P2.50mm
- R1, R2, R3, R4, R5, R6, U2, U4: moved to B.Cu
- U1: value ESP32-WROOM-32 -> ESP32-WROOM; footprint RF_Module:ESP32-WROOM-32 -> custom-footprint:ESP32-WROOM; moved to B.Cu
- moved R6 166.3 mm to (110.2, 53.8), turned to 90 degrees
- moved U4 161.9 mm to (111.5, 72.6), turned to -90 degrees
- moved C3 161.1 mm to (108.5, 44.5)
- moved U3 144.9 mm to (108.7, 57.7), turned to 90 degrees
- moved C4 144.9 mm to (104.9, 73.4), turned to 90 degrees
- moved C5 136.9 mm to (118.1, 73.3), turned to 90 degrees
- moved R7 136.9 mm to (112.5, 64.8)
- moved R5 126.9 mm to (136.1, 79.6), turned to 90 degrees
- moved R3 115.8 mm to (148.8, 70.9), turned to 180 degrees
- moved SW3 111.9 mm to (152.1, 76.7)
- moved D1 111.6 mm to (141.5, 94.0)
- moved Q1 111.4 mm to (136.7, 84.3), turned to 180 degrees
- moved R4 108.1 mm to (141.0, 86.4), turned to -90 degrees
- moved K1 100.9 mm to (133.9, 71.9), turned to 180 degrees
- moved RV1 98.8 mm to (153.6, 66.8), turned to 180 degrees
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Connections:
- net /VAC-OUT2 renamed /VAC-OUT1
- U1 pad 15: GND -> unconnected-(U1-Pad15)
- U1 pad 31: MOSI -> MISO
- U1 pad 39: GND -> unconnected-(U1-Pad39)
Routing:
- net GND: track 0.00 -> 254.3 mm, vias 0 -> 2
- net AC: track 0.00 -> 138.2 mm
- net +3V3: track 0.00 -> 131.9 mm, vias 0 -> 1
- net /AC_SENS_IN_1: track 0.00 -> 113.8 mm
- net +5V: track 0.00 -> 66.2 mm
- net VAC: track 0.00 -> 62.1 mm
- net Button_EN: track 0.00 -> 59.1 mm
- net SCL_RTC: track 0.00 -> 54.8 mm, vias 0 -> 2
- net SDA_RTC: track 0.00 -> 53.2 mm, vias 0 -> 2
- net /VAC-OUT1: track 0.00 -> 51.1 mm
- net Net-(D1-Pad1): track 0.00 -> 47.9 mm
- net Button_boot: track 0.00 -> 43.5 mm, vias 0 -> 1
- net OUT1: track 0.00 -> 38.7 mm, vias 0 -> 2
- net RST_LAN: track 0.00 -> 37.9 mm, vias 0 -> 1
- net MOSI: track 0.00 -> 37.4 mm
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Other:
- board outline added: 71.1 x 58.7 mm
