File: Hardware/Wireless Switch.kicad_sch (KiCad schematic)
At the start: 28 parts, among them J1 Uploader, J2 DC_INPUT, J3 OUTPUT1, J4 RTC_CON, K1 G3MB-202PDC5, Q1 BC547, SW1 BOOT, SW2 RESET, SW3 MODE, U1 ESP32-WROOM-32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

Commit message: route pcb
Parts:
- removed U1: ESP32-WROOM-32, RF_Module:ESP32-WROOM-32, symbol RF_Module:ESP32-WROOM-32
- added J5: AC_INPUT, TerminalBlock:TerminalBlock_Wuerth_691311400102_P7.62mm, symbol Connector:Conn_01x02_Female
- added U1: ESP32-WROOM, custom-footprint:ESP32-WROOM, symbol mainboardV2-rescue:ESP32-WROOM-ESP32-footprints-Shem-Lib
- C4: footprint Capacitor_SMD:CP_Elec_4x3.9 -> custom-footprint:CP_Radial_Tantal_D5.0mm_P2.50mm
- C5: value 10uf -> 22uf; footprint Capacitor_SMD:CP_Elec_4x3.9 -> custom-footprint:CP_Radial_Tantal_D5.0mm_P2.50mm
Connections:
- net +3V3: now also U1.2 (3V3)
- net AC: now also J5.1 (Pin_1)
- net Button_EN: now also U1.3 (EN)
- net Button_boot: now also U1.25 (IO0)
- net CLK: now also U1.30 (IO18)
- net GND: now also U1.1 (GND), U1.38 (GND)
- net MISO: now also U1.31 (IO19)
- net MOSI: now also U1.37 (IO23)
- net OUT1: now also U1.29 (IO5)
- net RST_LAN: now also U1.13 (IO14)
- net RX_Uploader: now also U1.34 (RXD0)
- net SCL_RTC: now also U1.36 (IO22)
- net SCS_LAN: now also U1.9 (IO33)
- net SDA_RTC: now also U1.33 (IO21)
- net SENSOR1: now also U1.27 (IO16)
- net TX_Uploader: now also U1.35 (TXD0)
- net VAC: now also J5.2 (Pin_2)
- no-connect marks 30 -> 33
